File: Ratt.kicad_pcb (KiCad board)
At the start: 2 copper layers, 80 x 70 mm, 17 parts, among them J2 MCP2551, J3 Conn_01x19, J4 ESP32 Connector, J7 Screw_Terminal_01x04, SW1 DriveMode(WE-42852752), SW2 SW_Coded_SH-7040, SW3 SW_Coded_SH-7040, U3 74HC4067

Commit message: Added capacity
Parts:
- added C1: C, Capacitor_SMD:C_0805_2012Metric_Pad1.18x1.45mm_HandSolder, F.Cu at (59.5, 49.4)
- added C2: C, Capacitor_SMD:C_0805_2012Metric_Pad1.18x1.45mm_HandSolder, F.Cu at (105.2, 88.8)
Routing:
- net Net-(U3-I12): track 18.4 -> 25.7 mm
- net Net-(J3-Pin_6): track 45.5 -> 49.4 mm
- net +5V: track 277.4 -> 280.8 mm
