File: Ratt.kicad_sch (KiCad schematic)
At the start: 15 parts, among them J2 MCP2551, J3 Conn_01x19, J4 ESP32 Connector, J7 Screw_Terminal_01x04, SW1 DriveMode(WE-42852752), SW2 SW_Coded_SH-7040, SW3 SW_Coded_SH-7040, U3 74HC4067

Commit message: Added capacity
Parts:
- added C1, C2: C, Capacitor_SMD:C_0805_2012Metric_Pad1.18x1.45mm_HandSolder, symbol Device:C
Connections:
- net +5V: now also C1.1, C2.1
- net GND: now also C1.2, C2.2
